File: split-clef.kicad_pcb (KiCad board)
At the start: 2 copper layers, 267.2 x 106.8 mm, 54 parts, among them J3 OLED

Commit message: v2
Parts:
- removed H1, H2, H3, H4, Ref** (x2): Val**, kicad-footprints:M2_HOLE_v2
- removed the J3 at (240.4, 136.3)
- removed the J3 at (185.9, 136.3)
- removed JET (x2): JST_PH_S2B-PH-K_1x02_P2.00mm_Horizontal, Connector_JST:JST_PH_S2B-PH-K_1x02_P2.00mm_Horizontal
- removed LS0, LS1, LS10, LS11, LS2, LS3, LS4, LS5, LS6, LS7, LS8, LS9, RS0, RS1, RS2, RS3 (x3), RS4, RS5, RS6, RS7, RS8, RS9: , kicad-footprints:ChocV1_V2_Hotswap
- removed M2_Mount (x4): , kicad-footprints:M2_HOLE_v2
- removed MCU (x2): SuperMini, split-clef:SuperMini NRF52840
- removed REF** (x8): Breakaway_Tabs, kicad-footprints:Breakaway_Tabs
- removed REF** (x2): Adafruit QSPI DIP Breakout Board, split-clef:Adafruit QSPI DIP Breakout Board
- removed RSW1 (x2): SW_PUSH, kicad-footprints:ResetSW_1side
- added ?: , , B.Cu at (190.3, 89.1)
- added ?: , , B.Cu at (249.6, 142.7)
- added ?: , , B.Cu at (249.5, 142.2)
- added ANT: ANTENNA_2450AT43B100E, split-clef:ANTENNA_2450AT43B100E, B.Cu at (172.0, 141.3)
- added ANT: ANTENNA_2450AT43B100E, split-clef:ANTENNA_2450AT43B100E, B.Cu at (236.8, 140.6)
- added C1: 1.0uF, Capacitor_SMD:C_0402_1005Metric, B.Cu at (190.8, 94.8)
- added C10: 100nF, Capacitor_SMD:C_0402_1005Metric, B.Cu at (180.3, 138.5)
- added C10: 100nF, Capacitor_SMD:C_0402_1005Metric, B.Cu at (184.8, 137.7)
- added C11: 100nF, Capacitor_SMD:C_0402_1005Metric, B.Cu at (177.0, 147.5)
- added C11: 100nF, Capacitor_SMD:C_0402_1005Metric, B.Cu at (177.1, 146.5)
- added C12: 1.0uF, Capacitor_SMD:C_0402_1005Metric, B.Cu at (185.8, 138.5)
- added C13: 4.7uF, Capacitor_SMD:C_0402_1005Metric, B.Cu at (188.3, 148.5)
- added C14: 10pF, Capacitor_SMD:C_0402_1005Metric, B.Cu at (241.8, 138.8)
- added C15: 10pF, Capacitor_SMD:C_0402_1005Metric, B.Cu at (245.9, 138.8)
- added C16: 18pF, Capacitor_SMD:C_0402_1005Metric, B.Cu at (252.4, 141.2)
- added C17: 18pF, Capacitor_SMD:C_0402_1005Metric, B.Cu at (252.4, 145.3)
- added C18: 100nF, Capacitor_SMD:C_0402_1005Metric, B.Cu at (246.8, 138.8)
- added C19: 1.0uf, Capacitor_SMD:C_0402_1005Metric, B.Cu at (246.6, 149.7)
- added C2: 2.2uf, Capacitor_SMD:C_0402_1005Metric, B.Cu at (189.2, 94.9)
- added C20: 100nF, Capacitor_SMD:C_0402_1005Metric, B.Cu at (244.0, 149.7)
- added C21: 4.7uF, Capacitor_SMD:C_0402_1005Metric, B.Cu at (249.5, 149.7)
- added C22: 1.0uF, Capacitor_SMD:C_0402_1005Metric, B.Cu at (252.4, 139.3)
- added C23: 4.7uF, Capacitor_SMD:C_0402_1005Metric, B.Cu at (252.4, 146.8)
- added C24: 4.7uF, Capacitor_SMD:C_0402_1005Metric, B.Cu at (252.4, 147.8)
- added C25: 4.7uF, Capacitor_SMD:C_0402_1005Metric, B.Cu at (248.6, 149.7)
- added C26: 0.8pF, Capacitor_SMD:C_0402_1005Metric, B.Cu at (241.8, 143.8)
- added C27: 1.0uF, Capacitor_SMD:C_0402_1005Metric, B.Cu at (241.3, 142.3)
- added C28: 100nF, Capacitor_SMD:C_0402_1005Metric, B.Cu at (242.5, 156.5)
- added C29: 0.8pF, Capacitor_SMD:C_0402_1005Metric, B.Cu at (176.9, 144.2)
- added C3: 10uF, Capacitor_SMD:C_0402_1005Metric, B.Cu at (194.5, 90.8)
- added C30: 0.5pF, Capacitor_SMD:C_0402_1005Metric, B.Cu at (174.9, 144.2)
- added C31: 0.2pF, Capacitor_SMD:C_0402_1005Metric, B.Cu at (173.9, 144.2)
- added C32: 4.7uF, Capacitor_SMD:C_0402_1005Metric, B.Cu at (188.3, 149.5)
- added C33: 1.0uF, Capacitor_SMD:C_0402_1005Metric, B.Cu at (177.0, 142.5)
- added C34: 100pF, Capacitor_SMD:C_0402_1005Metric, B.Cu at (177.0, 141.5)
- added C35: 100nF, Capacitor_SMD:C_0402_1005Metric, B.Cu at (188.1, 140.5)
- added C36: 0.5pF, Capacitor_SMD:C_0402_1005Metric, B.Cu at (239.8, 143.8)
- added C37: 100pF, Capacitor_SMD:C_0402_1005Metric, B.Cu at (241.3, 140.2)
- added C37: 100pF, Capacitor_SMD:C_0402_1005Metric, B.Cu at (249.4, 138.6)
- added C38: 4.7uF, Capacitor_SMD:C_0402_1005Metric, B.Cu at (186.2, 149.5)
- added C39: 4.7uF, Capacitor_SMD:C_0402_1005Metric, B.Cu at (185.3, 149.5)
- added C4: 10uF, Capacitor_SMD:C_0402_1005Metric, B.Cu at (186.3, 92.3)
- added C40: 1.0uf, Capacitor_SMD:C_0402_1005Metric, B.Cu at (181.9, 150.4)
- added C41: 100nF, Capacitor_SMD:C_0402_1005Metric, B.Cu at (170.0, 151.8)
- added C42: 0.2pF, Capacitor_SMD:C_0402_1005Metric, B.Cu at (238.8, 143.8)
- added C43: 100nF, Capacitor_SMD:C_0402_1005Metric, B.Cu at (252.4, 140.2)
- added C44: 1.0uF, Capacitor_SMD:C_0402_1005Metric, B.Cu at (239.0, 90.7)
- added C45: 2.2uf, Capacitor_SMD:C_0402_1005Metric, B.Cu at (240.4, 87.5)
- added C46: 10uF, Capacitor_SMD:C_0402_1005Metric, B.Cu at (236.2, 95.7)
- added C47: 10uF, Capacitor_SMD:C_0402_1005Metric, B.Cu at (235.7, 88.5)
- added C48: 10uF, Capacitor_SMD:C_0402_1005Metric, B.Cu at (231.7, 95.1)
- added C5: 10uF, Capacitor_SMD:C_0402_1005Metric, B.Cu at (187.1, 87.0)
- added C6: 10pF, Capacitor_SMD:C_0402_1005Metric, B.Cu at (177.1, 140.0)
- added C7: 10pF, Capacitor_SMD:C_0402_1005Metric, B.Cu at (178.5, 138.0)
- added C8: 18pF, Capacitor_SMD:C_0402_1005Metric, B.Cu at (189.9, 144.2)
- added C9: 18pF, Capacitor_SMD:C_0402_1005Metric, B.Cu at (188.3, 146.3)
- added D1: SMAJ5.0A, Diode_SMD:D_SMA, B.Cu at (184.0, 90.5)
- added D2: LED, LED_SMD:LED_0402_1005Metric, B.Cu at (184.3, 149.5)
- added D3: SMAJ5.0A, Diode_SMD:D_SMA, B.Cu at (243.1, 90.7)
- added D4: LED, LED_SMD:LED_0402_1005Metric, B.Cu at (230.7, 150.2)
- added J1: USB_C_Receptacle_USB2.0_16P, Connector_USB:USB_C_Receptacle_GCT_USB4105-xx-A_16P_TopMnt_Horizontal, B.Cu at (176.9, 89.1)
- added J2: Battery Connector, Connector_JST:JST_PH_S2B-PH-K_1x02_P2.00mm_Horizontal, B.Cu at (166.2, 88.8)
- added J3: OLED header, kicad-footprints:OLED_v2, F.Cu at (159.0, 92.2)
- added J4: USB_C_Receptacle_USB2.0_16P, Connector_USB:USB_C_Receptacle_GCT_USB4105-xx-A_16P_TopMnt_Horizontal, B.Cu at (250.4, 89.7)
- added J5: OLED header, kicad-footprints:OLED_v2, F.Cu at (267.2, 92.8)
- added J6: Battery Connector, Connector_JST:JST_PH_S2B-PH-K_1x02_P2.00mm_Horizontal, B.Cu at (261.9, 89.5)
- added L1: 2.2uH, Inductor_SMD:L_0805_2012Metric, B.Cu at (187.0, 89.6)
- added L2: 4.7nH, Inductor_SMD:L_0402_1005Metric, B.Cu at (240.8, 143.8)
- added L3: 4.7nH, Inductor_SMD:L_0402_1005Metric, B.Cu at (175.9, 144.2)
- added L4: 2.2uH, Inductor_SMD:L_0805_2012Metric, B.Cu at (233.9, 95.6)
- added LK0: SW_Push, kicad-footprints:ChocV1_V2_Hotswap, F.Cu at (90.1, 113.8)
- added LK1: SW_Push, kicad-footprints:ChocV1_V2_Hotswap, F.Cu at (109.1, 113.8)
- added LK10: SW_Push, kicad-footprints:ChocV1_V2_Hotswap, F.Cu at (166.1, 126.8)
- added LK11: SW_Push, kicad-footprints:ChocV1_V2_Hotswap, F.Cu at (185.2, 126.8)
- added LK12: SW_Push, kicad-footprints:ChocV1_V2_Hotswap, F.Cu at (159.9, 166.8)
- added LK13: SW_Push, kicad-footprints:ChocV1_V2_Hotswap, F.Cu at (179.0, 166.8)
- added LK14: SW_Push, kicad-footprints:ChocV1_V2_Hotswap, F.Cu at (198.0, 166.8)
- added LK2: SW_Push, kicad-footprints:ChocV1_V2_Hotswap, F.Cu at (128.1, 107.8)
- added LK3: SW_Push, kicad-footprints:ChocV1_V2_Hotswap, F.Cu at (147.1, 102.8)
- added LK4: SW_Push, kicad-footprints:ChocV1_V2_Hotswap, F.Cu at (166.1, 108.8)
- added LK5: SW_Push, kicad-footprints:ChocV1_V2_Hotswap, F.Cu at (185.2, 108.8)
- added LK6: SW_Push, kicad-footprints:ChocV1_V2_Hotswap, F.Cu at (90.1, 131.8)
- added LK7: SW_Push, kicad-footprints:ChocV1_V2_Hotswap, F.Cu at (109.1, 131.8)
- added LK8: SW_Push, kicad-footprints:ChocV1_V2_Hotswap, F.Cu at (128.1, 125.8)
- added LK9: SW_Push, kicad-footprints:ChocV1_V2_Hotswap, F.Cu at (147.1, 120.8)
- added R1: 5.1K, Resistor_SMD:R_0603_1608Metric, B.Cu at (173.4, 96.3)
- added R2: 5.1K, Resistor_SMD:R_0603_1608Metric, B.Cu at (179.3, 96.3)
- added R3: 1k, Resistor_SMD:R_0402_1005Metric, B.Cu at (195.7, 151.3)
- added R4: 1k5, Resistor_SMD:R_0402_1005Metric, B.Cu at (194.1, 92.9)
- added R5: 5.1K, Resistor_SMD:R_0603_1608Metric, B.Cu at (248.4, 96.0)
- added R6: 5.1K, Resistor_SMD:R_0603_1608Metric, B.Cu at (253.0, 96.0)
- added R7: 1k5, Resistor_SMD:R_0402_1005Metric, B.Cu at (237.2, 88.4)
- added R8: 1k, Resistor_SMD:R_0402_1005Metric, B.Cu at (231.8, 150.2)
- added RK0: SW_Push, kicad-footprints:ChocV1_V2_Hotswap, F.Cu at (241.0, 108.8)
- added RK1: SW_Push, kicad-footprints:ChocV1_V2_Hotswap, F.Cu at (260.2, 108.8)
- added RK10: SW_Push, kicad-footprints:ChocV1_V2_Hotswap, F.Cu at (317.2, 131.8)
- added RK11: SW_Push, kicad-footprints:ChocV1_V2_Hotswap, F.Cu at (336.2, 131.8)
- added RK12: SW_Push, kicad-footprints:ChocV1_V2_Hotswap, F.Cu at (228.2, 166.8)
- added RK13: SW_Push, kicad-footprints:ChocV1_V2_Hotswap, F.Cu at (247.2, 166.8)
- added RK14: SW_Push, kicad-footprints:ChocV1_V2_Hotswap, F.Cu at (266.2, 166.8)
- added RK2: SW_Push, kicad-footprints:ChocV1_V2_Hotswap, F.Cu at (279.2, 102.8)
- added RK3: SW_Push, kicad-footprints:ChocV1_V2_Hotswap, F.Cu at (298.2, 107.8)
- added RK4: SW_Push, kicad-footprints:ChocV1_V2_Hotswap, F.Cu at (317.2, 113.8)
- added RK5: SW_Push, kicad-footprints:ChocV1_V2_Hotswap, F.Cu at (336.2, 113.8)
- added RK6: SW_Push, kicad-footprints:ChocV1_V2_Hotswap, F.Cu at (241.0, 126.8)
- added RK7: SW_Push, kicad-footprints:ChocV1_V2_Hotswap, F.Cu at (260.2, 126.8)
- added RK8: SW_Push, kicad-footprints:ChocV1_V2_Hotswap, F.Cu at (279.2, 120.8)
- added RK9: SW_Push, kicad-footprints:ChocV1_V2_Hotswap, F.Cu at (298.2, 125.8)
- added SW16: Reset Button, split-clef:SW_TS-1088-AR02016, B.Cu at (194.5, 146.7)
- added SW32: Reset Button, split-clef:SW_TS-1088-AR02016, B.Cu at (231.7, 144.9)
- added U1: TPD4E05U06DQAR, Package_SON:USON-10_2.5x1.0mm_P0.5mm, B.Cu at (176.6, 95.7)
- added U2: nPM1100-QDXX, Package_DFN_QFN:QFN-24-1EP_4x4mm_P0.5mm_EP2.6x2.6mm_ThermalVias, B.Cu at (190.5, 91.0)
- added U3: nRF52840-QIXX, Package_DFN_QFN:Nordic_AQFN-73-1EP_7x7mm_P0.5mm, B.Cu at (182.6, 144.0)
- added U4: TPD4E05U06DQAR, Package_SON:USON-10_2.5x1.0mm_P0.5mm, B.Cu at (250.7, 95.5)
- added U5: W25Q128JVS, Package_SO:SOIC-8_5.3x5.3mm_P1.27mm, B.Cu at (175.2, 153.4)
- added U6: nRF52840-QIXX, Package_DFN_QFN:Nordic_AQFN-73-1EP_7x7mm_P0.5mm, B.Cu at (246.8, 144.2)
- added U7: W25Q128JVS, Package_SO:SOIC-8_5.3x5.3mm_P1.27mm, B.Cu at (238.6, 153.4)
- added U8: nPM1100-QDXX, Package_DFN_QFN:QFN-24-1EP_4x4mm_P0.5mm_EP2.6x2.6mm_ThermalVias, B.Cu at (235.9, 92.1)
- added Y1: 32MHz, Crystal:Crystal_SMD_2016-4Pin_2.0x1.6mm, B.Cu at (176.5, 138.2)
- added Y2: 32.768kHz, Crystal:Crystal_SMD_2012-2Pin_2.0x1.2mm, B.Cu at (188.2, 144.3)
- added Y3: 32MHz, Crystal:Crystal_SMD_2016-4Pin_2.0x1.6mm, B.Cu at (243.8, 138.4)
- added Y4: 32.768kHz, Crystal:Crystal_SMD_2012-2Pin_2.0x1.2mm, B.Cu at (252.4, 143.3)
- moved LOGO 94.6 mm to (243.3, 66.1)
- moved LOGO 20.9 mm to (215.1, 142.6)
Routing:
- net left: track 312.2 -> 0.00 mm
- net right: track 265.1 -> 0.00 mm, vias 2 -> 0
- net /VDD_NRF: track 0.00 -> 158.2 mm, vias 0 -> 7
- net /VDD_NRF-R: track 0.00 -> 155.7 mm, vias 0 -> 7
- net RK4: track 131.0 -> 0.00 mm
- net R-GND: track 130.6 -> 0.00 mm, vias 28 -> 0
- net /KEY5-R: track 0.00 -> 121.7 mm, vias 0 -> 2
- net LK5: track 120.0 -> 0.00 mm, vias 1 -> 0
- net /KEY11-R: track 0.00 -> 114.3 mm, vias 0 -> 2
- net RK9: track 113.2 -> 0.00 mm
- net RK3: track 108.9 -> 0.00 mm
- net GND: track 113.3 -> 5.70 mm, vias 23 -> 2
- net /D+: track 0.00 -> 106.2 mm, vias 0 -> 6
- net /KEY0: track 0.00 -> 105.6 mm, vias 0 -> 2
- net LK0: track 104.8 -> 0.00 mm, vias 1 -> 0
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- added copper zone on B.Cu, net GND2
- added copper zone on F.Cu, net GND2
- removed copper zone on B.Cu, net R-GND
- removed copper zone on F.Cu, net R-GND
Other:
- outline, holes or cut-outs redrawn
- board text removed: "+"
- board text removed: "GND"

Commit message: v2 finished, need to generate prods files
Parts:
- removed ? (x3): , 
- removed the C10 at (184.8, 137.7)
- removed the C11 at (177.1, 146.5)
- moved D2 11.3 mm to (195.4, 151.3)
- moved R3 1.38 mm to (194.3, 151.3), turned to 90 degrees
Connections:
- net DEC4_6-R renamed /DEC4_6-R
- C24 pad 1: Net-(U6-VDDH) -> /VDD_NRF-R
- C38 pad 1: /VDDH -> /VDD_NRF
- U3 pad M2: /KEY10 -> unconnected-(U3-P0.07-PadM2)
- U3 pad N1: /KEY11 -> unconnected-(U3-P0.08-PadN1)
- U3 pad N24: /VDD_NRF -> /Net-(C37-Pad1)
- U3 pad Y2: /VDDH -> /VDD_NRF
- U6 pad AD16: (no net) -> unconnected-(U6-P0.20-PadAD16)
- U6 pad AD20: (no net) -> unconnected-(U6-P0.24-PadAD20)
- U6 pad G1: /KEY7-R -> unconnected-(U6-P0.26-PadG1)
- U6 pad M2: (no net) -> unconnected-(U6-P0.07-PadM2)
- U6 pad T2: (no net) -> unconnected-(U6-P0.11-PadT2)
- U6 pad W24: (no net) -> unconnected-(U6-P1.02-PadW24)
- U6 pad Y2: Net-(U6-VDDH) -> /VDD_NRF-R
- U6 pad Y23: (no net) -> unconnected-(U6-P1.01-PadY23)
Routing:
- net VBUS-R: track 42.3 -> 120.7 mm, vias 0 -> 2
- net VBUS: track 13.0 -> 84.5 mm, vias 2 -> 6
- net GND2: track 0.77 -> 29.5 mm, vias 0 -> 2443
- net GND: track 5.70 -> 18.5 mm, vias 2 -> 2321
- net Net-(D2-K): track 13.8 -> 1.07 mm, vias 2 -> 0
- net /VDD_NRF-R: track 155.7 -> 160.8 mm, vias 7 -> 8
- net /VDDH: track 3.34 -> 0.00 mm, vias 2 -> 0
- net /VDD_NRF: track 158.2 -> 159.2 mm, vias 7 -> 9
- net Net-(U6-P0.01): track 4.88 -> 4.89 mm, vias 1 -> 2
- net Net-(U6-P0.00): track 4.58 -> 4.57 mm, vias 1 -> 2
- net /VSYS: vias 2 -> 3
Other:
- board text added: "{ "ViaStitching": "0.2", "stitch_zone_0": { "HSpacing": "1.27", "VSpacing": "1.17", "HOffset": "0", "VOffset": "0", "Clearance": "0.2", "Randomize": false } }"
- board text added: "{ "ViaStitching": "0.2", "stitch_zone_0": { "HSpacing": "1.27", "VSpacing": "1.27", "HOffset": "0", "VOffset": "0", "Clearance": "0.2", "Randomize": false } }"
