File: split-clef.kicad_sch (KiCad schematic)
At the start: 0 parts

Commit message: v1.0
Parts:
- added SW1, SW10, SW11, SW12, SW13, SW14, SW15, SW16, SW17, SW18, SW19, SW2, SW20, SW21, SW22, SW23, SW24, SW3, SW4, SW5, SW6, SW7, SW8, SW9: SW_Push, symbol Switch:SW_Push
- added U2: ~, symbol split-clef:0.9_OLED
- added U3: ~, symbol split-clef:W25Q128
- added leftMCU, rightMCU: ~, symbol split-clef:SuperMini_NRF52840
Connections:
- new net CLK: leftMCU. (P0.09)
- new net GND: U2. (SDA), U3. (G), leftMCU. (P0.09)
- new net I00: U3. (G), leftMCU. (P0.09)
- new net I01: U3. (G), leftMCU. (P0.09)
- new net KEY0: SW1.1, SW13.1, leftMCU. (P0.09), rightMCU. (P0.09)
- new net KEY1: SW15.1, SW2.1, leftMCU. (P0.09), rightMCU. (P0.09)
- new net KEY10: SW11.1, SW23.1, leftMCU. (P0.09), rightMCU. (P0.09)
- new net KEY11: SW12.1, SW24.1, leftMCU. (P0.09), rightMCU. (P0.09)
- new net KEY2: SW17.1, SW3.1, leftMCU. (P0.09), rightMCU. (P0.09)
- new net KEY3: SW19.1, SW4.1, leftMCU. (P0.09), rightMCU. (P0.09)
- new net KEY4: SW21.1, SW5.1, leftMCU. (P0.09), rightMCU. (P0.09)
- new net KEY5: SW14.1, SW6.1, leftMCU. (P0.09), rightMCU. (P0.09)
- new net KEY6: SW16.1, SW7.1, leftMCU. (P0.09), rightMCU. (P0.09)
- new net KEY7: SW18.1, SW8.1, leftMCU. (P0.09), rightMCU. (P0.09)
- new net KEY8: SW20.1, SW9.1, leftMCU. (P0.09), rightMCU. (P0.09)
- new net KEY9: SW10.1, SW22.1, leftMCU. (P0.09), rightMCU. (P0.09)
- new net SCL: U2. (SDA), leftMCU. (P0.09)
- new net SDA: U2. (SDA), leftMCU. (P0.09)
- new net VCC: U2. (SDA), U3. (G), leftMCU. (P0.09)
- new net left: SW1.2, SW10.2, SW11.2, SW12.2, SW2.2, SW3.2, SW4.2, SW5.2, SW6.2, SW7.2, SW8.2, SW9.2, leftMCU. (P0.09)
- new net right: SW13.2, SW14.2, SW15.2, SW16.2, SW17.2, SW18.2, SW19.2, SW20.2, SW21.2, SW22.2, SW23.2, SW24.2, rightMCU. (P0.09)

Commit message: v2
Parts:
- removed SW13, SW14, SW15, SW17, SW18, SW19, SW20, SW21, SW22, SW23, SW24: SW_Push, symbol Switch:SW_Push
- removed U2: ~, symbol split-clef:0.9_OLED
- removed U3: ~, symbol split-clef:W25Q128
- removed leftMCU, rightMCU: ~, symbol split-clef:SuperMini_NRF52840
- added BT1, BT2: Battery_Cell, symbol Device:Battery_Cell
- added C1, C12, C22, C27, C33, C44: 1.0uF, Capacitor_SMD:C_0402_1005Metric, symbol Device:C
- added C10, C11, C18, C20, C28, C35, C41, C43: 100nF, Capacitor_SMD:C_0402_1005Metric, symbol Device:C
- added C13, C21, C23, C24, C25, C32, C38, C39: 4.7uF, Capacitor_SMD:C_0402_1005Metric, symbol Device:C
- added C14, C15, C6, C7: 10pF, Capacitor_SMD:C_0402_1005Metric, symbol Device:C
- added C16, C17, C8, C9: 18pF, Capacitor_SMD:C_0402_1005Metric, symbol Device:C
- added C19, C40: 1.0uf, Capacitor_SMD:C_0402_1005Metric, symbol Device:C
- added C2, C45: 2.2uf, Capacitor_SMD:C_0402_1005Metric, symbol Device:C
- added C26, C29: 0.8pF, Capacitor_SMD:C_0402_1005Metric, symbol Device:C
- added C3, C4, C46, C47, C48, C5: 10uF, Capacitor_SMD:C_0402_1005Metric, symbol Device:C
- added C30, C36: 0.5pF, Capacitor_SMD:C_0402_1005Metric, symbol Device:C
- added C31, C42: 0.2pF, Capacitor_SMD:C_0402_1005Metric, symbol Device:C
- added C34, C37: 100pF, Capacitor_SMD:C_0402_1005Metric, symbol Device:C
- added D1, D3: SMAJ5.0A, Diode_SMD:D_SMA, symbol Diode:SMAJ5.0A
- added D2, D4: LED, LED_SMD:LED_0402_1005Metric, symbol Device:LED
- added J1, J4: USB_C_Receptacle_USB2.0_16P, Connector_USB:USB_C_Receptacle_GCT_USB4105-xx-A_16P_TopMnt_Horizontal, symbol Connector:USB_C_Receptacle_USB2.0_16P
- added J2, J6: Battery Connector, Connector_JST:JST_PH_S2B-PH-K_1x02_P2.00mm_Horizontal, symbol Connector:Conn_01x02_Socket
- added J3, J5: OLED header, kicad-footprints:OLED_v2, symbol Connector_Generic:Conn_01x04
- added L1, L4: 2.2uH, Inductor_SMD:L_0805_2012Metric, symbol Device:L
- added L2, L3: 4.7nH, Inductor_SMD:L_0402_1005Metric, symbol Device:L
- added LK12, LK13, LK14, RK0, RK1, RK10, RK11, RK12, RK13, RK14, RK2, RK3, RK4, RK5, RK6, RK7, RK8, RK9: SW_Push, kicad-footprints:ChocV1_V2_Hotswap, symbol Switch:SW_Push
- added R1, R2, R5, R6: 5.1K, Resistor_SMD:R_0603_1608Metric, symbol Device:R
- added R3, R8: 1k, Resistor_SMD:R_0402_1005Metric, symbol Device:R
- added R4, R7: 1k5, Resistor_SMD:R_0402_1005Metric, symbol Device:R
- added SW32: Reset Button, split-clef:SW_TS-1088-AR02016, symbol Switch:SW_Push
- added U1, U4: TPD4E05U06DQAR, Package_SON:USON-10_2.5x1.0mm_P0.5mm, symbol Power_Protection:TPD4EUSB30
- added U2, U8: nPM1100-QDXX, Package_DFN_QFN:QFN-24-1EP_4x4mm_P0.5mm_EP2.6x2.6mm_ThermalVias, symbol PCM_nordic-lib-kicad-npm:nPM1100-QDXX
- added U3, U6: nRF52840-QIXX, Package_DFN_QFN:Nordic_AQFN-73-1EP_7x7mm_P0.5mm, symbol PCM_nordic-lib-kicad-nrf52:nRF52840-QIXX
- added U5, U7: W25Q128JVS, Package_SO:SOIC-8_5.3x5.3mm_P1.27mm, symbol Memory_Flash:W25Q128JVS
- added Y1, Y3: 32MHz, Crystal:Crystal_SMD_2016-4Pin_2.0x1.6mm, symbol Device:Crystal
- added Y2, Y4: 32.768kHz, Crystal:Crystal_SMD_2012-2Pin_2.0x1.2mm, symbol Device:Crystal
- LK0: renamed from SW1; footprint (none) -> kicad-footprints:ChocV1_V2_Hotswap
- LK1: renamed from SW2; footprint (none) -> kicad-footprints:ChocV1_V2_Hotswap
- LK10: renamed from SW11; footprint (none) -> kicad-footprints:ChocV1_V2_Hotswap
- LK11: renamed from SW12; footprint (none) -> kicad-footprints:ChocV1_V2_Hotswap
- LK2: renamed from SW3; footprint (none) -> kicad-footprints:ChocV1_V2_Hotswap
- LK3: renamed from SW4; footprint (none) -> kicad-footprints:ChocV1_V2_Hotswap
- LK4: renamed from SW5; footprint (none) -> kicad-footprints:ChocV1_V2_Hotswap
- LK5: renamed from SW6; footprint (none) -> kicad-footprints:ChocV1_V2_Hotswap
- LK6: renamed from SW7; footprint (none) -> kicad-footprints:ChocV1_V2_Hotswap
- LK7: renamed from SW8; footprint (none) -> kicad-footprints:ChocV1_V2_Hotswap
- LK8: renamed from SW9; footprint (none) -> kicad-footprints:ChocV1_V2_Hotswap
- LK9: renamed from SW10; footprint (none) -> kicad-footprints:ChocV1_V2_Hotswap
- SW16: value SW_Push -> Reset Button; footprint (none) -> split-clef:SW_TS-1088-AR02016
Connections:
- net left is gone; now on net GND: LK0.2, LK1.2, LK10.2, LK11.2, LK2.2, LK3.2, LK4.2, LK5.2, LK6.2, LK7.2, LK8.2, LK9.2
- net right is gone; now on net GND: SW16.2
- net GND: now also BT2.2 (-), C1.2, C10.2, C11.2, C12.2, C13.2, C2.2, C29.2, C3.2, C30.2, C31.2, C32.2, C33.2, C34.2, C35.2, C38.2, C39.2, C4.2, C40.2, C41.1, C5.2, C6.1, C7.1, C8.1, C9.1, J1.A1 (GND), J1.A12 (GND), J1.B1 (GND), J1.B12 (GND), J1.S1 (SHIELD), J2.1 (Pin_1), J3.4 (Pin_4), LK12.2, LK13.2, LK14.2, R1.2, R2.2, R3.2, R4.2, U1.3 (GND), U1.8 (GND), U2.11 (SHPHLD), U2.23 (PVSS), U2.25 (AVSS), U2.4 (AVSS), U3.B7 (VSS), U3.EP (VSS), U3.F23 (VSS_PA), U5.4 (GND)
- net KEY0: now also U3.U24 (P1.04)
- net KEY1: now also U3.P23 (P1.07)
- net KEY10: now also U3.A20 (P1.10), U3.M2 (P0.07)
- net KEY11: now also U3.L1 (P0.06), U3.N1 (P0.08)
- net KEY2: now also U3.J24 (P0.10)
- net KEY3: now also U3.B19 (P1.11)
- net KEY4: now also U3.G1 (P0.26)
- net KEY5: now also U3.J1 (P0.04)
- net KEY6: now also U3.W24 (P1.02); no longer SW16.1
- net KEY7: now also U3.R24 (P1.06)
- net KEY8: now also U3.L24 (P0.09)
- net KEY9: now also U3.B17 (P1.12)
- net SCL: now also J3.2 (Pin_2), U3.A14 (P1.15)
- net SDA: now also J3.1 (Pin_1), U3.A16 (P1.13)
- new net: C32.1, U3.AC5 (DECUSB)
- new net: C29.1, L3.1, U3.H23 (ANT)
- new net: L1.2, U2.22 (SW)
- new net: C26.1, L2.1, U6.H23 (ANT)
- new net: D4.1 (K), R8.1
- new net: R4.1, U2.12 (ICHG)
- new net: C4.1, U2.21 (DEC)
- new net: C46.1, U8.21 (DEC)
- new net: C16.2, U6.D2 (P0.00), Y4.2
- new net: C15.2, U6.A23 (XC2), Y3.1
- new net: C25.1, U6.AC5 (DECUSB)
- new net: C14.2, U6.B24 (XC1), Y3.2
- new net: C43.1, U6.C1 (DEC1)
- new net: C37.1, U6.D23 (DEC3)
- new net: C17.2, U6.F2 (P0.01), Y4.1
- new net: C24.1, U6.Y2 (VDDH)
- new net: D3.2 (A2), J4.A4 (VBUS), J4.A9 (VBUS), J4.B4 (VBUS), J4.B9 (VBUS)
- new net: R7.1, U8.12 (ICHG)
- new net: J4.B5 (CC2), R6.1
- new net: D1.2 (A2), J1.A4 (VBUS), J1.A9 (VBUS), J1.B4 (VBUS), J1.B9 (VBUS)
- new net: J1.A5 (CC1), R1.1
- new net: J1.B5 (CC2), R2.1
- new net: J4.A5 (CC1), R5.1
- new net: L4.2, U8.22 (SW)
- new net: D2.1 (K), R3.1
- new net ANT: C30.1, C31.1, L3.2
- new net ANT-R: C36.1, C42.1, L2.2
- new net CHG: U2.8 (CHG), U3.A10 (P0.29)
- new net CHG-R: U6.R24 (P1.06), U8.8 (CHG)
- new net D+: J1.A6 (D+), J1.B6 (D+), U1.1 (D1+), U1.10 (NC), U1.4 (D2+), U1.7 (NC), U2.20 (D+), U3.AD6 (D+)
- new net D+R: J4.A6 (D+), J4.B6 (D+), U4.1 (D1+), U4.10 (NC), U4.4 (D2+), U4.7 (NC), U6.AD6 (D+), U8.20 (D+)
- new net D-: J1.A7 (D-), J1.B7 (D-), U1.2 (D1-), U1.5 (D2-), U1.6 (NC), U1.9 (NC), U2.19 (D-), U3.AD4 (D-)
- new net D-R: J4.A7 (D-), J4.B7 (D-), U4.2 (D1-), U4.5 (D2-), U4.6 (NC), U4.9 (NC), U6.AD4 (D-), U8.19 (D-)
- new net DEC1: C35.1, U3.C1 (DEC1)
- new net DEC3: C34.1, U3.D23 (DEC3)
- new net DEC4_6: C33.1, U3.B5 (DEC4), U3.E24 (DEC6)
- new net DEC4_6-R: C27.1, U6.B5 (DEC4), U6.E24 (DEC6)
- new net ERR: U2.10 (ERR), U3.A12 (P0.02)
- new net ERR-R: U6.U24 (P1.04), U8.10 (ERR)
- new net FCLK: U3.AC15 (P0.19), U5.6 (CLK)
- new net FCLK-R: U6.AC15 (P0.19), U7.6 (CLK)
- new net GND2: BT1.2 (-), C14.1, C15.1, C16.1, C17.1, C18.2, C19.2, C20.2, C21.2, C22.2, C23.2, C24.2, C25.2, C26.2, C27.2, C28.2, C36.2, C37.2, C42.2, C43.2, C44.2, C45.2, C46.2, C47.2, C48.2, J4.A1 (GND), J4.A12 (GND), J4.B1 (GND), J4.B12 (GND), J4.S1 (SHIELD), J5.4 (Pin_4), J6.1 (Pin_1), R5.2, R6.2, R7.2, R8.2, RK0.2, RK1.2, RK10.2, RK11.2, RK12.2, RK13.2, RK14.2, RK2.2, RK3.2, RK4.2, RK5.2, RK6.2, RK7.2, RK8.2, RK9.2, SW32.2, U4.3 (GND), U4.8 (GND), U6.B7 (VSS), U6.EP (VSS), U6.F23 (VSS_PA), U7.4 (GND), U8.11 (SHPHLD), U8.23 (PVSS), U8.25 (AVSS), U8.4 (AVSS)
- new net IO-0: U3.AC19 (P0.23), U5.5 (DI/IO_{0})
- new net IO-0-R: U6.AD18 (P0.22), U7.5 (DI/IO_{0})
- new net IO-1: U3.AD18 (P0.22), U5.2 (DO/IO_{1})
- new net IO-1-R: U6.AC19 (P0.23), U7.2 (DO/IO_{1})
- new net IO-2: U3.AC17 (P0.21), U5.3 (~{WP}/IO_{2})
- new net IO-2-R: U6.AC17 (P0.21), U7.3 (~{WP}/IO_{2})
- new net IO-3: U3.AD22 (P1.00), U5.7 (~{HOLD}/~{RESET}/IO_{3})
- new net IO-3-R: U6.AD22 (P1.00), U7.7 (~{HOLD}/~{RESET}/IO_{3})
- new net ISET: U2.5 (ISET), U3.U1 (P0.12)
- new net ISET-R: U6.J24 (P0.10), U8.5 (ISET)
- new net KEY0-R: RK0.1, U6.A20 (P1.10)
- new net KEY1-R: RK1.1, U6.A16 (P1.13)
- new net KEY10-R: RK10.1, U6.N1 (P0.08)
- new net KEY11-R: RK11.1, U6.U1 (P0.12)
- new net KEY12: LK12.1, U3.AD12 (P0.17)
- new net KEY12-R: RK12.1, U6.AD12 (P0.17)
- new net KEY13: LK13.1, U3.AD10 (P0.15)
- new net KEY13-R: RK13.1, U6.AD10 (P0.15)
- new net KEY14: LK14.1, U3.AD8 (P0.13)
- new net KEY14-R: RK14.1, U6.AD8 (P0.13)
- new net KEY2-R: RK2.1, U6.A12 (P0.02)
- new net KEY3-R: RK3.1, U6.J1 (P0.04)
- new net KEY4-R: RK4.1, U6.L1 (P0.06)
- new net KEY5-R: RK5.1, U6.R1 (P1.09)
- new net KEY6-R: RK6.1, U6.A18 (DEC2)
- new net KEY7-R: RK7.1, U6.A14 (P1.15), U6.G1 (P0.26)
- new net KEY8-R: RK8.1, U6.B13 (P0.03)
- new net KEY9-R: RK9.1, U6.H2 (P0.27)
- new net MODE: U2.7 (MODE), U3.A8 (P0.31)
- new net MODE-R: U6.L24 (P0.09), U8.7 (MODE)
- new net Net-(C37-Pad1): U3.N24 (DEC5)
- new net Net-(C38-Pad1): U3.A18 (DEC2)
- new net RST: SW16.1, U3.AC13 (~{RESET}), U5.1 (~{CS})
- new net RST-R: SW32.1, U6.AC13 (~{RESET}), U7.1 (~{CS})
- new net SCL-R: J5.2 (Pin_2), U6.A8 (P0.31)
- new net SDA-R: J5.1 (Pin_1), U6.A10 (P0.29)
- new net VBAT: BT2.1 (+), C1.1, J2.2 (Pin_2), U2.15 (VBAT)
- new net VBAT-R: BT1.1 (+), C44.1, J6.2 (Pin_2), U8.15 (VBAT)
- new net VBUS: C2.1, C39.1, D1.1 (A1), D2.2 (A), U2.17 (VBUS), U3.AD2 (VBUS)
- new net VBUS-R: C21.1, C45.1, D3.1 (A1), D4.2 (A), U6.AD2 (VBUS), U8.17 (VBUS)
- new net VDDH: C38.1, U3.Y2 (VDDH)
- new net VDDH-R: C18.1, C19.1, C20.1, C22.1, C23.1, C28.1, C48.1, J5.3 (Pin_3), L4.1, U6.A22 (VDD), U6.AD14 (VDD), U6.AD23 (VDD), U6.B1 (VDD), U6.W1 (VDD), U7.8 (VCC), U8.1 (VOUTB)
- new net VDD_NRF: C10.1, C11.1, C12.1, C13.1, C40.1, C41.2, C5.1, J3.3 (Pin_3), L1.1, U2.1 (VOUTB), U3.A22 (VDD), U3.AD14 (VDD), U3.AD23 (VDD), U3.B1 (VDD), U3.W1 (VDD), U5.8 (VCC)
- new net VSYS: C3.1, U2.16 (VSYS), U2.2 (VOUTBSET1), U2.3 (VOUTBSET0), U2.9 (VTERMSET)
- new net VSYS-R: C47.1, U8.16 (VSYS), U8.2 (VOUTBSET1), U8.3 (VOUTBSET0), U8.9 (VTERMSET)
- new net XC1: C6.2, U3.B24 (XC1), Y1.2
- new net XC2: C7.2, U3.A23 (XC2), Y1.1
- new net XL1: C8.2, U3.D2 (P0.00), Y2.2
- new net XL2: C9.2, U3.F2 (P0.01), Y2.1
- no-connect marks 0 -> 67
Other:
- note added: "Charge controller"
- note added: "Charge controller left"
- note added: "ERC Power flags"
- note added: "JST Battery Connector"
- note added: "Micro controller (NRF52840-QIAA) Left"
- note added: "Micro controller (NRF52840-QIAA) Right"
- note added: "QSPI Flash"
- note added: "USB-C"
- note added: "USB-C left"
- moved on the sheet: LK0, LK1, LK10, LK11, LK2, LK3, LK4, LK5, LK6, LK7, LK8, LK9

Commit message: v2 finished, need to generate prods files
Connections:
- net VDDH is gone; now on net VDD_NRF: C38.1, U3.Y2 (VDDH)
- net VDDH-R is gone; now on net VDD_NRF-R: C18.1, C19.1, C20.1, C22.1, C23.1, C28.1, C48.1, J5.3 (Pin_3), L4.1, U6.A22 (VDD), U6.AD14 (VDD), U6.AD23 (VDD), U6.B1 (VDD), U6.W1 (VDD), U7.8 (VCC), U8.1 (VOUTB)
- net KEY10: no longer U3.M2 (P0.07)
- net KEY11: no longer U3.N1 (P0.08)
- net KEY7-R: no longer U6.G1 (P0.26)
- net VDD_NRF-R: now reaches C24.1, U6.Y2 (VDDH)
- no-connect marks 67 -> 70
Changed lines of the file:
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@@
 	)
 	(junction
-		(at 590.55 496.57)
-		(diameter 0)
-		(color 0 0 0 0)
-	)
-	(junction
 		(at 271.78 463.55)
 		(diameter 0)
@@
 	)
 	(junction
-		(at 359.41 497.84)
-		(diameter 0)
-		(color 0 0 0 0)
-	)
-	(junction
 		(at 566.42 496.57)
 		(diameter 0)
@@
 	)
 	(no_connect
+		(at 64.77 421.64)
+	)
+	(no_connect
 		(at 746.76 477.52)
 	)
@@
 	)
 	(no_connect
+		(at 680.72 429.26)
+	)
+	(no_connect
 		(at 105.41 335.28)
 	)
@@
 	)
 	(no_connect
+		(at 130.81 457.2)
+	)
+	(no_connect
 		(at 64.77 469.9)
 	)
@@
 	(wire
 		(pts
-			(xy 368.3 501.65) (xy 359.41 501.65)
-		)
-		(stroke
-			(width 0)
-			(type default)
-		)
-	)
-	(wire
-		(pts
 			(xy 109.22 200.66) (xy 116.84 200.66)
 		)
@@
 	(wire
 		(pts
-			(xy 359.41 497.84) (xy 368.3 497.84)
-		)
-		(stroke
-			(width 0)
-			(type default)
-		)
-	)
-	(wire
-		(pts
 			(xy 330.2 381) (xy 330.2 382.27)
 		)
@@
 	(wire
 		(pts
-			(xy 590.55 496.57) (xy 599.44 496.57)
+			(xy 580.39 496.57) (xy 599.44 496.57)
 		)
 		(stroke
@@
 	(wire
 		(pts
-			(xy 359.41 501.65) (xy 359.41 497.84)
-		)
-		(stroke
-			(width 0)
-			(type default)
-		)
-	)
-	(wire
-		(pts
 			(xy 347.98 361.95) (xy 347.98 360.68)
 		)
@@
 	(wire
 		(pts
-			(xy 746.76 337.82) (xy 770.89 337.82)
-		)
-		(stroke
-			(width 0)
-			(type default)
-		)
-	)
-	(wire
-		(pts
 			(xy 49.53 370.84) (xy 58.42 370.84)
 		)
@@
 	(wire
 		(pts
-			(xy 681.99 294.64) (xy 681.99 299.72)
+			(xy 746.76 337.82) (xy 770.89 337.82)
 		)
 		(stroke
@@
 	(wire
 		(pts
-			(xy 693.42 492.76) (xy 693.42 497.84)
+			(xy 681.99 294.64) (xy 681.99 299.72)
 		)
 		(stroke
@@
 	(wire
 		(pts
-			(xy 64.77 368.3) (xy 58.42 368.3)
+			(xy 693.42 492.76) (xy 693.42 497.84)
 		)
 		(stroke
@@
 	(wire
 		(pts
-			(xy 711.2 492.76) (xy 711.2 497.84)
+			(xy 64.77 368.3) (xy 58.42 368.3)
 		)
 		(stroke
@@
 	(wire
 		(pts
-			(xy 359.41 497.84) (xy 349.25 497.84)
+			(xy 711.2 492.76) (xy 711.2 497.84)
 		)
 		(stroke
@@
 	(wire
 		(pts
-			(xy 93.98 335.28) (xy 93.98 320.04)
+			(xy 349.25 497.84) (xy 368.3 497.84)
 		)
 		(stroke
@@
 	(wire
 		(pts
-			(xy 590.55 496.57) (xy 580.39 496.57)
+			(xy 93.98 335.28) (xy 93.98 320.04)
 		)
 		(stroke
@@
 	(wire
 		(pts
-			(xy 590.55 500.38) (xy 590.55 496.57)
-		)
-		(stroke
-			(width 0)
-			(type default)
-		)
-	)
-	(wire
-		(pts
 			(xy 64.77 363.22) (xy 58.42 363.22)
 		)
@@
 	(wire
 		(pts
-			(xy 599.44 500.38) (xy 590.55 500.38)
-		)
-		(stroke
-			(width 0)
-			(type default)
-		)
-	)
-	(wire
-		(pts
 			(xy 510.54 389.89) (xy 511.81 389.89)
 		)
@@
 		)
 	)
-	(label "VDD_NRF-R"
-		(at 695.96 495.3 0)
-		(effects
-			(font
-				(size 1.27 1.27)
-			)
-			(justify left bottom)
-		)
-	)
 	(label "RST"
 		(at 152.4 518.16 180)
@@
 	)
 	(label "DEC4_6-R"
-		(at 746.76 337.82 0)
+		(at 753.11 337.82 0)
 		(effects
 			(font
@@
 		)
 	)
-	(label "VDD_NRF"
-		(at 368.3 501.65 0)
-		(effects
-			(font
-				(size 1.27 1.27)
-			)
-			(justify left bottom)
-		)
-	)
 	(label "XL2"
 		(at 49.53 391.16 270)
@@
 	)
 	(label "DEC4_6-R"
-		(at 746.76 337.82 0)
+		(at 753.11 337.82 0)
 		(effects
 			(font
@@
 		)
 	)
+	(label "DEC4_6-R"
+		(at 753.11 332.74 0)
+		(effects
+			(font
+				(size 1.27 1.27)
+			)
+			(justify left bottom)
+		)
+	)
 	(label "XC2"
 		(at 49.53 368.3 270)
@@
 		)
 	)
-	(label "DEC4_6-R"
-		(at 746.76 337.82 0)
+	(label "VDD_NRF-R"
+		(at 699.77 492.76 0)
 		(effects
 			(font
@@
 		)
 	)
-	(label "VDD_NRF-R"
-		(at 676.91 492.76 0)
+	(label "DEC4_6-R"
+		(at 753.11 337.82 0)
 		(effects
 			(font
@@
 		)
 	)
-	(label "VDDH"
+	(label "VDD_NRF"
 		(at 102.87 325.12 0)
 		(effects
@@
 		)
 	)
-	(label "KEY11"
-		(at 64.77 421.64 180)
-		(effects
-			(font
-				(size 1.27 1.27)
-			)
-			(justify right bottom)
-		)
-	)
 	(label "MODE"
 		(at 64.77 467.36 180)
@@
 		)
 	)
+	(label "VDD_NRF-R"
+		(at 676.91 492.76 0)
+		(effects
+			(font
+				(size 1.27 1.27)
+			)
+			(justify left bottom)
+		)
+	)
 	(label "KEY2-R"
 		(at 530.86 351.79 90)
@@
 		)
 	)
-	(label "KEY10"
-		(at 130.81 457.2 0)
-		(effects
-			(font
-				(size 1.27 1.27)
-			)
-			(justify left bottom)
-		)
-	)
-	(label "VDDH-R"
-		(at 599.44 500.38 0)
+	(label "VDD_NRF-R"
+		(at 698.5 497.84 0)
 		(effects
 			(font
@@
 		)
 	)
+	(label "VDD_NRF-R"
+		(at 718.82 299.72 0)
+		(effects
+			(font
+				(size 1.27 1.27)
+			)
+			(justify left bottom)
+		)
+	)
 	(label "KEY13"
 		(at 64.77 429.26 180)
@@
 		)
 	)
-	(label "VDD_NRF-R"
-		(at 688.34 497.84 0)
-		(effects
-			(font
-				(size 1.27 1.27)
-			)
-			(justify left bottom)
-		)
-	)
 	(label "VBAT"
 		(at 358.14 449.58 0)
@@
 		)
 	)
-	(label "KEY7-R"
-		(at 680.72 429.26 180)
-		(effects
-			(font
-				(size 1.27 1.27)
-			)
-			(justify right bottom)
-		)
-	)
 	(label "D-"
 		(at 109.22 210.82 0)
@@
 		)
 	)
-	(label "VDD_NRF-R"
-		(at 701.04 492.76 0)
-		(effects
-			(font
-				(size 1.27 1.27)
-			)
-			(justify left bottom)
-		)
-	)
 	(label "KEY2-R"
 		(at 680.72 383.54 180)
@@
 		)
 	)
+	(label "VDD_NRF-R"
+		(at 689.61 497.84 0)
+		(effects
+			(font
+				(size 1.27 1.27)
+			)
+			(justify left bottom)
+		)
+	)
